File: SevSeg-Shield/SevSeg-Shield-v10.brd (EAGLE design)
At the start: 59.7 x 53.3 mm, 5 parts, among them U2 ARDUINO_SHIELD

Commit message: Updated the footprint of the display.
Proto worked but the footprint was not quite right. This version should
work a lot better.
Connections:
- removed net VCC: U2.5V
Changed lines of the file:
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@@
 <wire x1="34.29" y1="2.54" x2="31.75" y2="2.54" width="0.254" layer="1"/>
-</signal>
-<signal name="VCC">
-<contactref element="U2" pad="5V"/>
 </signal>
 <signal name="ARST">
